File: e-ink-a-sketch.kicad_sch (KiCad schematic)
At the start: 7 parts, among them J1 EPD, J2 IMU, M1 Motor_DC, SW1 RotaryEncoder_Switch, SW2 RotaryEncoder_Switch, U1 XIAO-ESP32-C3-SMD

Commit message: added boxes
Other:
- note added: "ENCODERS"
- note added: "EPD"
- note added: "IMU"
- note added: "MCU"
- note added: "VIBRATION MOTOR"
- moved on the sheet: J2, M1
Changed lines of the file:
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@@
 	(generator_version "10.0")
 	(paper "A4")
+	(rectangle
+		(start 177.8 83.82)
+		(end 221.615 128.27)
+		(stroke
+			(width 0.254)
+			(type solid)
+		)
+		(fill
+			(type none)
+		)
+	)
+	(rectangle
+		(start 99.06 51.435)
+		(end 176.53 135.89)
+		(stroke
+			(width 0.254)
+			(type solid)
+		)
+		(fill
+			(type none)
+		)
+	)
+	(rectangle
+		(start 62.865 105.41)
+		(end 97.79 135.89)
+		(stroke
+			(width 0.254)
+			(type solid)
+		)
+		(fill
+			(type none)
+		)
+	)
+	(rectangle
+		(start 60.96 73.025)
+		(end 97.79 104.14)
+		(stroke
+			(width 0.254)
+			(type solid)
+		)
+		(fill
+			(type none)
+		)
+	)
+	(rectangle
+		(start 62.23 41.275)
+		(end 97.79 71.755)
+		(stroke
+			(width 0.254)
+			(type solid)
+		)
+		(fill
+			(type none)
+		)
+	)
+	(text "EPD"
+		(exclude_from_sim no)
+		(at 63.119 74.93 0)
+		(effects
+			(font
+				(size 1.27 1.27)
+			)
+		)
+	)
+	(text "VIBRATION MOTOR"
+		(exclude_from_sim no)
+		(at 72.136 107.696 0)
+		(effects
+			(font
+				(size 1.27 1.27)
+			)
+		)
+	)
+	(text "ENCODERS"
+		(exclude_from_sim no)
+		(at 183.896 85.852 0)
+		(effects
+			(font
+				(size 1.27 1.27)
+			)
+		)
+	)
+	(text "IMU"
+		(exclude_from_sim no)
+		(at 64.389 43.18 0)
+		(effects
+			(font
+				(size 1.27 1.27)
+			)
+		)
+	)
+	(text "MCU"
+		(exclude_from_sim no)
+		(at 102.108 53.594 0)
+		(effects
+			(font
+				(size 1.27 1.27)
+			)
+		)
+	)
 	(no_connect
-		(at 85.725 62.23)
+		(at 76.2 62.23)
 	)
 	(no_connect
-		(at 85.725 59.69)
+		(at 76.2 59.69)
 	)
 	(no_connect
@@
 	)
 	(no_connect
-		(at 85.725 64.77)
+		(at 76.2 64.77)
 	)
 	(no_connect
@@
 	(wire
 		(pts
-			(xy 69.85 123.19) (xy 82.55 123.19)
+			(xy 66.04 111.76) (xy 78.74 111.76)
 		)
 		(stroke
@@
 	(wire
 		(pts
-			(xy 94.615 54.61) (xy 85.725 54.61)
+			(xy 85.09 54.61) (xy 76.2 54.61)
 		)
 		(stroke
@@
 	(wire
 		(pts
-			(xy 98.425 49.53) (xy 85.725 49.53)
+			(xy 88.9 49.53) (xy 76.2 49.53)
 		)
 		(stroke
@@
 	(wire
 		(pts
-			(xy 82.55 135.89) (xy 82.55 137.16)
+			(xy 78.74 124.46) (xy 78.74 125.73)
 		)
 		(stroke
@@
 	(wire
 		(pts
-			(xy 98.425 52.07) (xy 85.725 52.07)
+			(xy 88.9 52.07) (xy 76.2 52.07)
 		)
 		(stroke
@@
 	(wire
 		(pts
-			(xy 94.615 57.15) (xy 85.725 57.15)
+			(xy 85.09 57.15) (xy 76.2 57.15)
 		)
 		(stroke
@@
 	(wire
 		(pts
-			(xy 94.615 67.31) (xy 85.725 67.31)
+			(xy 85.09 67.31) (xy 76.2 67.31)
 		)
 		(stroke
@@
 	)
 	(label "IMU_SDA"
-		(at 94.615 57.15 180)
+		(at 85.09 57.15 180)
 		(effects
 			(font
@@
 	)
 	(label "IMU_SCL"
-		(at 94.615 54.61 180)
+		(at 85.09 54.61 180)
 		(effects
 			(font
@@
 	)
 	(label "MOTOR_PWM"
-		(at 69.85 123.19 0)
+		(at 66.04 111.76 0)
 		(effects
 			(font
@@
 	)
 	(label "IMU_INT"
-		(at 94.615 67.31 180)
+		(at 85.09 67.31 180)
 		(effects
 			(font
@@
 	(symbol
 		(lib_id "power:GND")
-		(at 98.425 52.07 0)
+		(at 88.9 52.07 0)
 		(unit 1)
 		(body_style 1)
@@
 		(dnp no)
 		(property "Reference" "#PWR012"
-			(at 98.425 58.42 0)
+			(at 88.9 58.42 0)
 			(hide yes)
 			(show_name no)
@@
 		)
 		(property "Value" "GND"
-			(at 101.981 53.848 0)
+			(at 92.456 53.848 0)
 			(show_name no)
 			(do_not_autoplace no)
@@
 		)
 		(property "Footprint" ""
-			(at 98.425 52.07 0)
+			(at 88.9 52.07 0)
 			(hide yes)
 			(show_name no)
@@
 		)
 		(property "Datasheet" ""
-			(at 98.425 52.07 0)
+			(at 88.9 52.07 0)
 			(hide yes)
 			(show_name no)
@@
 		)
 		(property "Description" "Power symbol creates a global label with name \"GND\" , ground"
-			(at 98.425 52.07 0)
+			(at 88.9 52.07 0)
 			(hide yes)
 			(show_name no)
@@
 	(symbol
 		(lib_id "power:GND")
-		(at 82.55 137.16 0)
+		(at 78.74 125.73 0)
 		(unit 1)
 		(body_style 1)
@@
 		(dnp no)
 		(property "Reference" "#PWR09"
-			(at 82.55 143.51 0)
+			(at 78.74 132.08 0)
 			(hide yes)
 			(show_name no)
@@
 		)
 		(property "Value" "GND"
-			(at 82.55 141.224 0)
+			(at 78.74 129.794 0)
 			(show_name no)
 			(do_not_autoplace no)
@@
 		)
 		(property "Footprint" ""
-			(at 82.55 137.16 0)
+			(at 78.74 125.73 0)
 			(hide yes)
 			(show_name no)
@@
 		)
 		(property "Datasheet" ""
-			(at 82.55 137.16 0)
+			(at 78.74 125.73 0)
 			(hide yes)
 			(show_name no)
@@
 		)
 		(property "Description" "Power symbol creates a global label with name \"GND\" , ground"
-			(at 82.55 137.16 0)
+			(at 78.74 125.73 0)
 			(hide yes)
 			(show_name no)
@@
 		(lib_name "Conn_01x08_Socket_1")
 		(lib_id "Connector:Conn_01x08_Socket")
-		(at 80.645 57.15 0)
+		(at 71.12 57.15 0)
 		(mirror y)
 		(unit 1)
@@
 		(dnp no)
 		(property "Reference" "J2"
-			(at 86.233 44.704 0)
+			(at 76.708 44.704 0)
 			(show_name no)
 			(do_not_autoplace no)
@@
 		)
 		(property "Value" "IMU"
-			(at 86.233 47.244 0)
+			(at 76.708 47.244 0)
 			(show_name no)
 			(do_not_autoplace no)
@@
 		)
 		(property "Footprint" ""
-			(at 80.645 57.15 0)
+			(at 71.12 57.15 0)
 			(hide yes)
 			(show_name no)
@@
 		)
 		(property "Datasheet" ""
-			(at 80.645 57.15 0)
+			(at 71.12 57.15 0)
 			(hide yes)
 			(show_name no)
@@
 		)
 		(property "Description" "Generic connector, single row, 01x08, script generated"
-			(at 80.645 57.15 0)
+			(at 71.12 57.15 0)
 			(hide yes)
 			(show_name no)
@@
 	(symbol
 		(lib_id "Motor:Motor_DC")
-		(at 82.55 128.27 0)
+		(at 78.74 116.84 0)
 		(unit 1)
 		(body_style 1)
@@
 		(fields_autoplaced yes)
 		(property "Reference" "M1"
-			(at 87.63 129.5399 0)
+			(at 83.82 118.1099 0)
 			(show_name no)
 			(do_not_autoplace no)
@@
 		)
 		(property "Value" "Motor_DC"
-			(at 87.63 132.0799 0)
+			(at 83.82 120.6499 0)
 			(show_name no)
 			(do_not_autoplace no)
@@
 		)
 		(property "Footprint" ""
-			(at 82.55 130.556 0)
+			(at 78.74 119.126 0)
 			(hide yes)
 			(show_name no)
@@
 		)
 		(property "Datasheet" ""
-			(at 82.55 130.556 0)
+			(at 78.74 119.126 0)
 			(hide yes)
 			(show_name no)
@@
 		)
 		(property "Description" "DC Motor"
-			(at 82.55 128.27 0)
+			(at 78.74 116.84 0)
 			(hide yes)
 			(show_name no)
@@
 	(symbol
 		(lib_id "power:+3V3")
-		(at 98.425 49.53 0)
+		(at 88.9 49.53 0)
 		(unit 1)
 		(body_style 1)
@@
 		(dnp no)
 		(property "Reference" "#PWR013"
-			(at 98.425 53.34 0)
+			(at 88.9 53.34 0)
 			(hide yes)
 			(show_name no)
@@
 		)
 		(property "Value" "+3V3"
-			(at 101.727 47.498 0)
+			(at 92.202 47.498 0)
 			(show_name no)
 			(do_not_autoplace no)
@@
 		)
 		(property "Footprint" ""
-			(at 98.425 49.53 0)
+			(at 88.9 49.53 0)
 			(hide yes)
 			(show_name no)
@@
 		)
 		(property "Datasheet" ""
-			(at 98.425 49.53 0)
+			(at 88.9 49.53 0)
 			(hide yes)
 			(show_name no)
@@
 		)
 		(property "Description" "Power symbol creates a global label with name \"+3V3\""
-			(at 98.425 49.53 0)
-			(hide yes)
-			(show_name no)
+			(at 88.9 49.53 0)
+			(hide yes)
+			(show_name no)
